File: pengendali-lampu-laci/rev02/pengendali lampu laci.kicad_pcb (KiCad board)
At the start: 2 copper layers, 50 x 64 mm, 18 parts, among them P1 Power

Commit message: Update lighting controller
Parts:
- removed VCC +5V: JUMPER3, Pin_Headers:Pin_Header_Straight_1x03
- added REF***: OSHW-Logo2_9.8x8mm_SilkScreen, Symbols:OSHW-Logo2_9.8x8mm_SilkScreen, B.Cu at (75.6, 74.3)
Connections:
- Arduino Nano pad 30: /VIN -> Net-(Arduino1-Pad30)
- C1 pad 1: VCC -> +5V
- P1 pad 1: VCC -> +5V
Routing:
- net /VIN: track 100.7 -> 0.00 mm
- net VCC: track 21.4 -> 0.00 mm
- net +5V: track 0.00 -> 11.4 mm
- net Net-(Hub2-Pad8): track 52.1 -> 41.4 mm
- net /In5: track 24.1 -> 28.0 mm
- net /In11: track 53.1 -> 49.9 mm
- net /In12: track 52.4 -> 49.7 mm
- net /In6: track 26.8 -> 28.8 mm
- net /In10: track 22.3 -> 23.8 mm
- net /In2: track 27.4 -> 26.2 mm
- net /In3: track 25.9 -> 25.1 mm
- net /In1: track 29.7 -> 29.0 mm
Other:
- board text added: "GND +5V"
- board text added: "fajran 2016"
- board text added: "lighting controller"
- board text added: "rev01"
- board text removed: "GND VCC"
