File: pengendali-lampu-laci/archived/01/pcb/pengendali lampu laci.sch (KiCad schematic (older format))
At the start: 15 parts, among them P1 Power

Commit message: Move archived
Parts:
- removed JP1: JUMPER, Pin_Headers:Pin_Header_Straight_1x02, symbol JUMPER
- P1: footprint Connect:bornier2 -> Connect:BARREL_JACK
Connections:
- net labels removed: VCC
- wire segments 84 -> 82
