File: lighting-controller/rev01/pengendali lampu laci.kicad_pcb (KiCad board)
At the start: 2 copper layers, 50 x 64 mm, 18 parts, among them P1 Power

Commit message: Update controller
Routing:
- net Net-(Hub2-Pad8): track 41.4 -> 49.9 mm
- net /Out4: track 13.2 -> 14.6 mm
- net /Out3: track 10.1 -> 11.5 mm
- net /Out2: track 7.72 -> 8.84 mm
- net Net-(Hub1-Pad8): track 35.8 -> 36.4 mm
