File: drawer-lighting/lampu-laci-dapur.sch (KiCad schematic (older format))
At the start: 6 parts, among them P1 InPort, P3 InPad, P4 OutPad

Commit message: Update connector pads
Parts:
- P3, P4: footprint Pad:FourPad_2.0mm -> Pad:FourPad_2.0mm_FrontPTH_Side
Changed lines of the file:
@@
 F 0 "P3" H 1000 3500 50  0000 C CNN
 F 1 "InPad" V 1100 3250 50  0000 C CNN
-F 2 "Pad:FourPad_2.0mm" H 1000 3250 50  0001 C CNN
+F 2 "Pad:FourPad_2.0mm_FrontPTH_Side" H 1000 3250 50  0001 C CNN
 F 3 "" H 1000 3250 50  0000 C CNN
 	1    1000 3250
@@
 $EndComp
 $Comp
-L GND #PWR09
+L GND #PWR07
 U 1 1 57AD223F
 P 1250 3450
-F 0 "#PWR09" H 1250 3200 50  0001 C CNN
+F 0 "#PWR07" H 1250 3200 50  0001 C CNN
 F 1 "GND" H 1250 3300 50  0000 C CNN
 F 2 "" H 1250 3450 50  0000 C CNN
@@
 $EndComp
 $Comp
-L +5V #PWR010
+L +5V #PWR08
 U 1 1 57AD2245
 P 1650 3250
-F 0 "#PWR010" H 1650 3100 50  0001 C CNN
+F 0 "#PWR08" H 1650 3100 50  0001 C CNN
 F 1 "+5V" H 1650 3390 50  0000 C CNN
 F 2 "" H 1650 3250 50  0000 C CNN
@@
 F 0 "P4" H 2150 3500 50  0000 C CNN
 F 1 "OutPad" V 2250 3250 50  0000 C CNN
-F 2 "Pad:FourPad_2.0mm" H 2150 3250 50  0001 C CNN
+F 2 "Pad:FourPad_2.0mm_FrontPTH_Side" H 2150 3250 50  0001 C CNN
 F 3 "" H 2150 3250 50  0000 C CNN
 	1    2150 3250
@@
 $EndComp
 $Comp
-L GND #PWR011
+L GND #PWR09
 U 1 1 57AD2259
 P 2400 3450
-F 0 "#PWR011" H 2400 3200 50  0001 C CNN
+F 0 "#PWR09" H 2400 3200 50  0001 C CNN
 F 1 "GND" H 2400 3300 50  0000 C CNN
 F 2 "" H 2400 3450 50  0000 C CNN
@@
 $EndComp
 $Comp
-L +5V #PWR012
+L +5V #PWR010
 U 1 1 57AD225F
 P 2800 3250
-F 0 "#PWR012" H 2800 3100 50  0001 C CNN
+F 0 "#PWR010" H 2800 3100 50  0001 C CNN
 F 1 "+5V" H 2800 3390 50  0000 C CNN
 F 2 "" H 2800 3250 50  0000 C CNN
