File: drawer-sensor/TCRT5000/r02/sensor-laci-dapur.kicad_pcb (KiCad board)
At the start: 2 copper layers, 45.7 x 29.5 mm, 10 parts, among them U1 1_Out

Commit message: Update sensor
Other:
- board text added: "FAJRAN 2016"
- board text added: "REV 02"
- board text removed: "fajran 2016"
- board text removed: "rev02"
Changed lines of the file:
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@@
     (thickness 1.6)
     (drawings 33)
-    (tracks 19)
+    (tracks 21)
     (zones 0)
     (modules 10)
@@
   (gr_line (start 116.332 86.36) (end 116.332 78.74) (angle 90) (layer Eco1.User) (width 0.2))
   (gr_line (start 116.332 116.84) (end 116.332 109.22) (angle 90) (layer Eco1.User) (width 0.2))
-  (gr_text rev02 (at 161.544 109.728) (layer F.SilkS)
-    (effects (font (size 1 1) (thickness 0.1)) (justify left))
-  )
-  (gr_text "fajran 2016" (at 137.414 109.728) (layer F.SilkS)
+  (gr_text "REV 02" (at 165.1 109.855) (layer F.SilkS)
+    (effects (font (size 1 1) (thickness 0.1)) (justify right))
+  )
+  (gr_text "FAJRAN 2016" (at 137.795 109.855) (layer F.SilkS)
     (effects (font (size 1 1) (thickness 0.1)) (justify left))
   )
@@
   (segment (start 136.95 101.898) (end 136.95 99.06) (width 0.25) (layer F.Cu) (net 2))
   (segment (start 137.922 102.87) (end 136.95 101.898) (width 0.25) (layer F.Cu) (net 2))
+  (segment (start 165.227 95.33) (end 165.227 95.374998) (width 0.25) (layer F.Cu) (net 3))
+  (segment (start 165.227 95.374998) (end 163.573998 97.028) (width 0.25) (layer F.Cu) (net 3))
+  (segment (start 163.573998 97.028) (end 156.464 97.028) (width 0.25) (layer F.Cu) (net 3))
   (segment (start 155.194 97.79) (end 155.702 97.79) (width 0.25) (layer F.Cu) (net 3))
-  (segment (start 155.702 97.79) (end 158.162 95.33) (width 0.25) (layer F.Cu) (net 3))
-  (segment (start 165.227 95.33) (end 158.162 95.33) (width 0.25) (layer F.Cu) (net 3))
+  (segment (start 155.702 97.79) (end 156.464 97.028) (width 0.25) (layer F.Cu) (net 3))
   (segment (start 153.384 97.79) (end 155.194 97.79) (width 0.25) (layer F.Cu) (net 3))
   (segment (start 165.227 97.83) (end 156.678 97.83) (width 0.25) (layer F.Cu) (net 5))

Commit message: Remove OSHW logo
Parts:
- removed REF***: OSHW-Logo2_9.8x8mm_SilkScreen, Symbols:OSHW-Logo2_9.8x8mm_SilkScreen
